File: PCB/modern-keyboard.kicad_sch (KiCad schematic)
At the start: 0 parts

Commit message: organization
Parts:
- added A1: RaspberryPi_Pico, Module:RaspberryPi_Pico_Common_THT, symbol MCU_Module:RaspberryPi_Pico_Extensive
- added D1, D10, D11, D12, D13, D14, D15, D16, D17, D18, D19, D2, D20, D21, D22, D23, D24, D25, D26, D27, D28, D29, D3, D30, D31, D32, D33, D34, D35, D36, D37, D38, D39, D4, D40, D41, D42, D43, D44, D45, D46, D47, D48, D49, D5, D50, D51, D52, D53, D54, D55, D56, D57, D58, D59, D6, D60, D61, D62, D63, D64, D65, D66, D67, D7, D8, D9: D, Diode_THT:D_DO-35_SOD27_P7.62mm_Horizontal, symbol Device:D
- added LED1, LED10, LED11, LED12, LED13, LED14, LED15, LED16, LED17, LED18, LED19, LED2, LED20, LED21, LED22, LED23, LED24, LED25, LED26, LED27, LED28, LED29, LED3, LED30, LED31, LED32, LED33, LED34, LED35, LED36, LED37, LED38, LED39, LED4, LED40, LED41, LED42, LED43, LED44, LED45, LED46, LED47, LED48, LED49, LED5, LED50, LED51, LED52, LED53, LED54, LED55, LED56, LED57, LED58, LED59, LED6, LED60, LED61, LED62, LED63, LED64, LED65, LED66, LED67, LED7, LED8, LED9: SK6812MINI-E, PCM_marbastlib-xp-gateron_lp:LED_KS33_6028R-ROT, symbol PCM_marbastlib-various:SK6812MINI-E
- added SW1, SW10, SW11, SW12, SW13, SW16, SW17, SW18, SW19, SW2, SW20, SW21, SW22, SW23, SW24, SW25, SW26, SW27, SW29, SW3, SW31, SW32, SW33, SW34, SW35, SW36, SW37, SW38, SW39, SW4, SW40, SW41, SW43, SW45, SW46, SW47, SW48, SW49, SW5, SW50, SW51, SW52, SW53, SW54, SW56, SW57, SW6, SW62, SW63, SW64, SW65, SW66, SW67, SW7, SW8, SW9: SW_Push_45deg, marbastlib-xp-gateron_lp:SW_KS33_HS_KS-2P02B01-02_HS_1u, symbol Switch:SW_Push_45deg
- added SW14: SW_Push_45deg, marbastlib-xp-gateron_lp:SW_KS33_HS_KS-2P02B01-02_HS_2u, symbol Switch:SW_Push_45deg
- added SW15, SW28: SW_Push_45deg, marbastlib-xp-gateron_lp:SW_KS33_HS_KS-2P02B01-02_1.5u, symbol Switch:SW_Push_45deg
- added SW30, SW55: SW_Push_45deg, marbastlib-xp-gateron_lp:SW_KS33_HS_KS-2P02B01-02_1.75u, symbol Switch:SW_Push_45deg
- added SW42, SW44: SW_Push_45deg, marbastlib-xp-gateron_lp:SW_KS33_HS_KS-2P02B01-02_HS_2.25u, symbol Switch:SW_Push_45deg
- added SW58, SW59, SW60: SW_Push_45deg, marbastlib-xp-gateron_lp:SW_KS33_HS_KS-2P02B01-02_1.25u, symbol Switch:SW_Push_45deg
- added SW61: SW_Push_45deg, marbastlib-xp-gateron_lp:SW_KS33_HS_KS-2P02B01-02_HS_6.25u, symbol Switch:SW_Push_45deg
- added SW83: RotaryEncoder_Switch, Rotary_Encoder:RotaryEncoder_Alps_EC11E-Switch_Vertical_H20mm, symbol Device:RotaryEncoder_Switch
Connections:
- new net: D33.2 (A), SW33.2
- new net: LED19.2 (DOUT), LED20.3 (DIN)
- new net: LED18.2 (DOUT), LED19.3 (DIN)
- new net: D24.2 (A), SW24.2
- new net: D43.2 (A), SW43.2
- new net: D51.2 (A), SW51.2
- new net: D5.2 (A), SW5.2
- new net: LED17.2 (DOUT), LED18.3 (DIN)
- new net: LED53.2 (DOUT), LED54.3 (DIN)
- new net: LED52.2 (DOUT), LED53.3 (DIN)
- new net: D57.2 (A), SW57.2
- new net: D29.2 (A), SW29.2
- new net: D66.2 (A), SW66.2
- new net: D15.2 (A), SW15.2
- new net: D62.2 (A), SW62.2
- new net: D13.2 (A), SW13.2
- new net: D35.2 (A), SW35.2
- new net: LED48.2 (DOUT), LED49.3 (DIN)
- new net: LED47.2 (DOUT), LED48.3 (DIN)
- new net: D10.2 (A), SW10.2
- new net: D52.2 (A), SW52.2
- new net: D12.2 (A), SW12.2
- new net: D41.2 (A), SW41.2
- new net: D32.2 (A), SW32.2
- new net: LED25.2 (DOUT), LED26.3 (DIN)
- new net: LED24.2 (DOUT), LED25.3 (DIN)
- new net: D61.2 (A), SW61.2
- new net: LED13.2 (DOUT), LED14.3 (DIN)
- new net: LED12.2 (DOUT), LED13.3 (DIN)
- new net: D11.2 (A), SW11.2
- new net: LED23.2 (DOUT), LED24.3 (DIN)
- new net: LED10.3 (DIN), LED9.2 (DOUT)
- new net: LED8.2 (DOUT), LED9.3 (DIN)
- new net: D60.2 (A), SW60.2
- new net: D67.2 (A), SW67.2
- new net: D31.2 (A), SW31.2
- new net: LED21.2 (DOUT), LED22.3 (DIN)
- new net: LED20.2 (DOUT), LED21.3 (DIN)
- new net: D46.2 (A), SW46.2
- new net: D49.2 (A), SW49.2
- new net: D36.2 (A), SW36.2
- new net: D45.2 (A), SW45.2
- new net: D58.2 (A), SW58.2
- new net: LED14.2 (DOUT), LED15.3 (DIN)
- new net: LED5.2 (DOUT), LED6.3 (DIN)
- new net: LED4.2 (DOUT), LED5.3 (DIN)
- new net: LED27.2 (DOUT), LED28.3 (DIN)
- new net: LED26.2 (DOUT), LED27.3 (DIN)
- new net: D20.2 (A), SW20.2
- new net: D7.2 (A), SW7.2
- new net: D14.2 (A), SW14.2
- new net: D64.2 (A), SW64.2
- new net: LED62.2 (DOUT), LED63.3 (DIN)
- new net: LED61.2 (DOUT), LED62.3 (DIN)
- new net: LED7.2 (DOUT), LED8.3 (DIN)
- new net: LED6.2 (DOUT), LED7.3 (DIN)
- new net: D21.2 (A), SW21.2
- new net: D59.2 (A), SW59.2
- new net: D19.2 (A), SW19.2
- new net: LED10.2 (DOUT), LED11.3 (DIN)
- new net: LED38.2 (DOUT), LED39.3 (DIN)
- new net: LED37.2 (DOUT), LED38.3 (DIN)
- new net: D16.2 (A), SW16.2
- new net: D38.2 (A), SW38.2
- new net: LED54.2 (DOUT), LED55.3 (DIN)
- new net: D56.2 (A), SW56.2
- new net: D54.2 (A), SW54.2
- new net: D9.2 (A), SW9.2
- new net: LED32.2 (DOUT), LED33.3 (DIN)
- new net: LED31.2 (DOUT), LED32.3 (DIN)
- new net: D53.2 (A), SW53.2
- new net: D4.2 (A), SW4.2
- new net: D18.2 (A), SW18.2
- new net: LED30.2 (DOUT), LED31.3 (DIN)
- new net: LED29.2 (DOUT), LED30.3 (DIN)
- new net: D47.2 (A), SW47.2
- new net: D28.2 (A), SW28.2
- new net: LED28.2 (DOUT), LED29.3 (DIN)
- new net: D34.2 (A), SW34.2
- new net: D55.2 (A), SW55.2
- new net: D6.2 (A), SW6.2
- new net: D30.2 (A), SW30.2
- new net: LED11.2 (DOUT), LED12.3 (DIN)
- new net: LED33.2 (DOUT), LED34.3 (DIN)
- new net: D42.2 (A), SW42.2
- new net: D27.2 (A), SW27.2
- new net: LED41.2 (DOUT), LED42.3 (DIN)
- new net: LED40.2 (DOUT), LED41.3 (DIN)
- new net: LED36.2 (DOUT), LED37.3 (DIN)
- new net: LED39.2 (DOUT), LED40.3 (DIN)
- new net: LED22.2 (DOUT), LED23.3 (DIN)
- new net: D1.2 (A), SW1.2
- new net: LED66.2 (DOUT), LED67.3 (DIN)
- new net: D22.2 (A), SW22.2
- new net: LED55.2 (DOUT), LED56.3 (DIN)
- new net: LED65.2 (DOUT), LED66.3 (DIN)
- new net: LED58.2 (DOUT), LED59.3 (DIN)
- new net: LED57.2 (DOUT), LED58.3 (DIN)
- new net: LED64.2 (DOUT), LED65.3 (DIN)
- new net: D8.2 (A), SW8.2
- new net: D65.2 (A), SW65.2
- new net: LED44.2 (DOUT), LED45.3 (DIN)
- new net: LED43.2 (DOUT), LED44.3 (DIN)
- new net: D48.2 (A), SW48.2
- new net: LED56.2 (DOUT), LED57.3 (DIN)
- new net: D2.2 (A), SW2.2
- new net: LED35.2 (DOUT), LED36.3 (DIN)
- new net: LED34.2 (DOUT), LED35.3 (DIN)
- new net: LED45.2 (DOUT), LED46.3 (DIN)
- new net: D25.2 (A), SW25.2
- new net: D40.2 (A), SW40.2
- new net: LED50.2 (DOUT), LED51.3 (DIN)
- new net: LED49.2 (DOUT), LED50.3 (DIN)
- new net: D39.2 (A), SW39.2
- new net: LED59.2 (DOUT), LED60.3 (DIN)
- new net: D23.2 (A), SW23.2
- new net: LED46.2 (DOUT), LED47.3 (DIN)
- new net: D26.2 (A), SW26.2
- new net: D3.2 (A), SW3.2
- new net: LED15.2 (DOUT), LED16.3 (DIN)
- new net: LED51.2 (DOUT), LED52.3 (DIN)
- new net: LED60.2 (DOUT), LED61.3 (DIN)
- new net: D50.2 (A), SW50.2
- new net: D37.2 (A), SW37.2
- new net: LED16.2 (DOUT), LED17.3 (DIN)
- new net: D17.2 (A), SW17.2
- new net: LED42.2 (DOUT), LED43.3 (DIN)
- new net: LED63.2 (DOUT), LED64.3 (DIN)
- new net: LED3.2 (DOUT), LED4.3 (DIN)
- new net: LED2.2 (DOUT), LED3.3 (DIN)
- new net: LED1.2 (DOUT), LED2.3 (DIN)
- new net: D44.2 (A), SW44.2
- new net: D63.2 (A), SW63.2
- new net +3V3: A1.37 (3V3_EN)
- new net +5V: A1.40 (VBUS), LED1.1 (VDD), LED10.1 (VDD), LED11.1 (VDD), LED12.1 (VDD), LED13.1 (VDD), LED14.1 (VDD), LED15.1 (VDD), LED16.1 (VDD), LED17.1 (VDD), LED18.1 (VDD), LED19.1 (VDD), LED2.1 (VDD), LED20.1 (VDD), LED21.1 (VDD), LED22.1 (VDD), LED23.1 (VDD), LED24.1 (VDD), LED25.1 (VDD), LED26.1 (VDD), LED27.1 (VDD), LED28.1 (VDD), LED29.1 (VDD), LED3.1 (VDD), LED30.1 (VDD), LED31.1 (VDD), LED32.1 (VDD), LED33.1 (VDD), LED34.1 (VDD), LED35.1 (VDD), LED36.1 (VDD), LED37.1 (VDD), LED38.1 (VDD), LED39.1 (VDD), LED4.1 (VDD), LED40.1 (VDD), LED41.1 (VDD), LED42.1 (VDD), LED43.1 (VDD), LED44.1 (VDD), LED45.1 (VDD), LED46.1 (VDD), LED47.1 (VDD), LED48.1 (VDD), LED49.1 (VDD), LED5.1 (VDD), LED50.1 (VDD), LED51.1 (VDD), LED52.1 (VDD), LED53.1 (VDD), LED54.1 (VDD), LED55.1 (VDD), LED56.1 (VDD), LED57.1 (VDD), LED58.1 (VDD), LED59.1 (VDD), LED6.1 (VDD), LED60.1 (VDD), LED61.1 (VDD), LED62.1 (VDD), LED63.1 (VDD), LED64.1 (VDD), LED65.1 (VDD), LED66.1 (VDD), LED67.1 (VDD), LED7.1 (VDD), LED8.1 (VDD), LED9.1 (VDD)
- new net Col 0: A1.1 (GPIO0), SW1.1, SW15.1, SW30.1, SW44.1, SW58.1
- new net Col 1: A1.2 (GPIO1), SW16.1, SW2.1, SW31.1, SW45.1, SW59.1
- new net Col 10: A1.14 (GPIO10), SW11.1, SW25.1, SW40.1, SW54.1, SW63.1
- new net Col 11: A1.15 (GPIO11), SW12.1, SW26.1, SW41.1, SW64.1
- new net Col 12: A1.16 (GPIO12), SW13.1, SW27.1, SW55.1, SW65.1
- new net Col 13: A1.17 (GPIO13), SW14.1, SW28.1, SW42.1, SW56.1, SW66.1
- new net Col 14: A1.19 (GPIO14), SW29.1, SW43.1, SW57.1, SW67.1, SW83.S2
- new net Col 2: A1.4 (GPIO2), SW17.1, SW3.1, SW32.1, SW46.1, SW60.1
- new net Col 3: A1.5 (GPIO3), SW18.1, SW33.1, SW4.1, SW47.1
- new net Col 4: A1.6 (GPIO4), SW19.1, SW34.1, SW48.1, SW5.1
- new net Col 5: A1.7 (GPIO5), SW20.1, SW35.1, SW49.1, SW6.1, SW61.1
- new net Col 6: A1.9 (GPIO6), SW21.1, SW36.1, SW50.1, SW7.1
- new net Col 7: A1.10 (GPIO7), SW22.1, SW37.1, SW51.1, SW8.1
- new net Col 8: A1.11 (GPIO8), SW23.1, SW38.1, SW52.1, SW9.1
- new net Col 9: A1.12 (GPIO9), SW10.1, SW24.1, SW39.1, SW53.1, SW62.1
- new net EC1A: A1.21 (GPIO16), SW83.A
- new net EC1B: A1.22 (GPIO17), SW83.B
- new net GND: A1.13 (GND), A1.18 (GND), A1.23 (GND), A1.28 (GND), A1.3 (GND), A1.38 (GND), A1.8 (GND), A1.D2 (GND), A1.TP1 (USB_GND), LED1.4 (VSS), LED10.4 (VSS), LED11.4 (VSS), LED12.4 (VSS), LED13.4 (VSS), LED14.4 (VSS), LED15.4 (VSS), LED16.4 (VSS), LED17.4 (VSS), LED18.4 (VSS), LED19.4 (VSS), LED2.4 (VSS), LED20.4 (VSS), LED21.4 (VSS), LED22.4 (VSS), LED23.4 (VSS), LED24.4 (VSS), LED25.4 (VSS), LED26.4 (VSS), LED27.4 (VSS), LED28.4 (VSS), LED29.4 (VSS), LED3.4 (VSS), LED30.4 (VSS), LED31.4 (VSS), LED32.4 (VSS), LED33.4 (VSS), LED34.4 (VSS), LED35.4 (VSS), LED36.4 (VSS), LED37.4 (VSS), LED38.4 (VSS), LED39.4 (VSS), LED4.4 (VSS), LED40.4 (VSS), LED41.4 (VSS), LED42.4 (VSS), LED43.4 (VSS), LED44.4 (VSS), LED45.4 (VSS), LED46.4 (VSS), LED47.4 (VSS), LED48.4 (VSS), LED49.4 (VSS), LED5.4 (VSS), LED50.4 (VSS), LED51.4 (VSS), LED52.4 (VSS), LED53.4 (VSS), LED54.4 (VSS), LED55.4 (VSS), LED56.4 (VSS), LED57.4 (VSS), LED58.4 (VSS), LED59.4 (VSS), LED6.4 (VSS), LED60.4 (VSS), LED61.4 (VSS), LED62.4 (VSS), LED63.4 (VSS), LED64.4 (VSS), LED65.4 (VSS), LED66.4 (VSS), LED67.4 (VSS), LED7.4 (VSS), LED8.4 (VSS), LED9.4 (VSS), SW83.C
- new net RGB: A1.20 (GPIO15), LED1.3 (DIN)
- new net Row 0: A1.24 (GPIO18), D1.1 (K), D10.1 (K), D11.1 (K), D12.1 (K), D13.1 (K), D14.1 (K), D2.1 (K), D3.1 (K), D4.1 (K), D5.1 (K), D6.1 (K), D7.1 (K), D8.1 (K), D9.1 (K), SW83.S1
- new net Row 1: A1.25 (GPIO19), D15.1 (K), D16.1 (K), D17.1 (K), D18.1 (K), D19.1 (K), D20.1 (K), D21.1 (K), D22.1 (K), D23.1 (K), D24.1 (K), D25.1 (K), D26.1 (K), D27.1 (K), D28.1 (K), D29.1 (K)
- new net Row 2: A1.26 (GPIO20), D30.1 (K), D31.1 (K), D32.1 (K), D33.1 (K), D34.1 (K), D35.1 (K), D36.1 (K), D37.1 (K), D38.1 (K), D39.1 (K), D40.1 (K), D41.1 (K), D42.1 (K), D43.1 (K)
- new net Row 3: A1.27 (GPIO21), D44.1 (K), D45.1 (K), D46.1 (K), D47.1 (K), D48.1 (K), D49.1 (K), D50.1 (K), D51.1 (K), D52.1 (K), D53.1 (K), D54.1 (K), D55.1 (K), D56.1 (K), D57.1 (K)
- new net Row 4: A1.29 (GPIO22), D58.1 (K), D59.1 (K), D60.1 (K), D61.1 (K), D62.1 (K), D63.1 (K), D64.1 (K), D65.1 (K), D66.1 (K), D67.1 (K)
- no-connect marks 0 -> 1

Commit message: final
Parts:
- added C1, C2, C3, C4, C5, C6, C7, C8: 2.2 uF, Capacitor_SMD:C_0805_2012Metric_Pad1.18x1.45mm_HandSolder, symbol Device:C
Connections:
- net +5V: now also C1.1, C2.1, C3.1, C4.1, C5.1, C6.1, C7.1, C8.1
- net GND: now also C1.2, C2.2, C3.2, C4.2, C5.2, C6.2, C7.2, C8.2
